File: USB_HGA22_V1/USB_HGA22_V1.kicad_sch (KiCad schematic)
At the start: 57 parts, among them J1 LSCO, J2 RTC_OUT1, J3V3 Conn_01x02, J5V0 Conn_01x02, Q1 BSS138DW, U1 STM32C071G8UxN, U2 LP5907MFX-3.3, U3 LM321LV, Y1 SSPT7F-9PF10-R

Commit message: Documentation uploaded.
Other:
- note added: "250-mA Ultra-Low-Noise Low-IQ LDO"
- note added: "AGC 10-10000"
- note added: "DCF77_Ferrite_Ant = 1.357 mH"
- note added: "DEBUG"
- note added: "LPF"
- note added: "Mixer"
- note added: "RF Amplifier"
- note added: "SERIAL1"
- note added: "SERIAL2"
- note added: "STMicroelectronics Arm Cortex-M0+ MCU, 64KB flash, 24KB RAM"
- note added: "Voltage Tests"
- moved on the sheet: C10, C11, C4, C6, C7, C8, C9, CC2, CF1, CF2, JSER1, JSER2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
